File: pcb/power/power.kicad_sch (KiCad schematic)
At the start: 40 parts

Commit message: Semifinish power and bulk
Parts:
- removed C1, C10, C11, C12, C13, C14, C15, C16, C17, C18, C19, C2, C20, C21, C22, C23, C24, C25, C26, C27, C28, C29, C3, C30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: 2u2, Capacitor_SMD:C_1206_3216Metric, symbol Device:C
