File: pcb/power/phase.kicad_sch (KiCad schematic)
At the start: 9 parts, among them J1 Conn_01x02_Pin, J4 Conn_01x02_Pin, J7 Conn_01x02_Pin, Q10 IPT015N10NF2S, Q2 IPT015N10NF2S, Q5 IPT015N10NF2S, Q6 IPT015N10NF2S

Commit message: Semifinish power and bulk
Parts:
- removed J1, J4, J7: Conn_01x02_Pin, Connector_PinHeader_2.54mm:PinHeader_2x01_P2.54mm_Vertical_SMD, symbol Connector:Conn_01x02_Pin
- added C1: 100n, Capacitor_SMD:C_0402_1005Metric, symbol Device:C
- added C10, C2, C3, C4, C5, C6, C7, C8, C9: 2u2, Capacitor_SMD:C_1206_3216Metric, symbol Device:C
- added J1: Conn_02x01, Connector_PinHeader_1.27mm:PinHeader_2x01_P1.27mm_Vertical_SMD, symbol Connector_Generic:Conn_02x01
- added J2: Conn_02x03_Odd_Even, Connector_PinHeader_1.27mm:PinHeader_2x03_P1.27mm_Vertical_SMD, symbol Connector_Generic:Conn_02x03_Odd_Even
- added R2: 1m, Resistor_SMD:R_2512_6332Metric, symbol Device:R
- added U1: INA181, Package_TO_SOT_SMD:SOT-23-6, symbol Amplifier_Current:INA181
- R1: footprint Resistor_SMD:R_4020_10251Metric -> Resistor_SMD:R_2512_6332Metric; LCSC (none) -> C5123666
- R3: renamed from R4; footprint Resistor_SMD:R_4020_10251Metric -> Resistor_SMD:R_2512_6332Metric; LCSC (none) -> C5123666
- renumbered Q6 to Q1, Q5 to Q2, Q2 to Q3, Q10 to Q4
Connections:
- net GH: now also J1.1 (Pin_1)
- net GL: now also J2.5 (Pin_5)
- net GND: now also C1.2, J2.4 (Pin_4), U1.2 (GND); no longer R1.2, R3.2
- net SH: now reaches Q3.2 (S), Q4.2 (S), R1.1, R3.1
- net SH: now also J2.3 (Pin_3), R2.1, U1.4 (-)
- net PH: now reaches Q1.2 (S), Q2.2 (S), Q3.3 (D), Q4.3 (D)
- net PH: now also J1.2 (Pin_2)
- net VDD renamed VBUS
- net VBUS: now also C10.1, C2.1, C3.1, C4.1, C5.1, C6.1, C7.1, C8.1, C9.1
- new net CUR: J2.6 (Pin_6), U1.1
- new net GNDPWR: C10.2, C2.2, C3.2, C4.2, C5.2, C6.2, C7.2, C8.2, C9.2, R1.2, R2.2, R3.2, U1.3 (+)
- new net VCC: C1.1, J2.2 (Pin_2), U1.6 (V+)
- new net VREF: J2.1 (Pin_1), U1.5 (REF)
Other:
- moved on the sheet: Q1, Q2, Q3, Q4, R3

Commit message: Save progress
Parts:
- removed J1: Conn_02x01, Connector_PinHeader_1.27mm:PinHeader_2x01_P1.27mm_Vertical_SMD, symbol Connector_Generic:Conn_02x01
- added J1: Conn_02x02_Odd_Even, Connector_PinHeader_1.27mm:PinHeader_2x02_P1.27mm_Vertical_SMD, symbol Connector_Generic:Conn_02x02_Odd_Even
- Q1, Q2, Q3, Q4: value IPT015N10NF2S -> SP010N01BGHTO; LCSC C19632811 -> C22385350
Connections:
- net GH: now also J1.3 (Pin_3), J1.4 (Pin_4)
- net PH: now also J1.1 (Pin_1), J1.2 (Pin_2)

Commit message: Update shunts
Parts:
- R1, R2, R3: footprint Resistor_SMD:R_2512_6332Metric -> Resistor_SMD:R_4020_10251Metric; LCSC C5123666 -> C2927603
Changed lines of the file:
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@@
 			)
 		)
-		(property "Footprint" "Resistor_SMD:R_2512_6332Metric"
+		(property "Footprint" "Resistor_SMD:R_4020_10251Metric"
 			(at 49.022 102.87 90)
 			(effects
@@
 			)
 		)
-		(property "LCSC" "C5123666"
+		(property "LCSC" "C2927603"
 			(at 50.8 102.87 0)
 			(effects
@@
 			)
 		)
-		(property "Footprint" "Resistor_SMD:R_2512_6332Metric"
+		(property "Footprint" "Resistor_SMD:R_4020_10251Metric"
 			(at 41.402 102.87 90)
 			(effects
@@
 			)
 		)
-		(property "LCSC" "C5123666"
+		(property "LCSC" "C2927603"
 			(at 43.18 102.87 0)
 			(effects
@@
 			)
 		)
-		(property "Footprint" "Resistor_SMD:R_2512_6332Metric"
+		(property "Footprint" "Resistor_SMD:R_4020_10251Metric"
 			(at 33.782 102.87 90)
 			(effects
@@
 			)
 		)
-		(property "LCSC" "C5123666"
+		(property "LCSC" "C2927603"
 			(at 35.56 102.87 0)
 			(effects

Commit message: Finish rev 1
Parts:
- removed Q1, Q2, Q3, Q4: SP010N01BGHTO, Package_TO_SOT_SMD:Infineon_PG-HSOF-8-1, symbol Transistor_FET:IPT015N10N5
- added Q1, Q2, Q3, Q4: SP010N01BGHTO, Package_TO_SOT_SMD:Infineon_PG-HSOF-8-1, symbol User_Symbols:SP010N01BGHTO
- C1: LCSC C1525 -> C307331
- R1, R2, R3: footprint Resistor_SMD:R_4020_10251Metric -> User_Footprints:R_Shunt_3921
Connections:
- net GH: now also Q1.1 (G), Q2.1 (G)
- net GL: now also Q3.1 (G), Q4.1 (G)
- net GNDPWR: no longer C10.2, C2.2, C3.2, C4.2, C5.2, C6.2, C7.2, C8.2, C9.2
- net PH: now also Q1.2 (S), Q2.2 (S), Q3.3 (D), Q4.3 (D)
- net SH: now also Q3.2 (S), Q4.2 (S)
- net VBUS: now also Q1.3 (D), Q2.3 (D)
- net GND renamed AGND
- net VCC renamed 3V3
- new net GNDRET: C10.2, C2.2, C3.2, C4.2, C5.2, C6.2, C7.2, C8.2, C9.2
Other:
- note added: "Connectors"
- note added: "Half Bridge + Shunt + Amplifier"
- note added: "High Freq Bypass Ceramics"
- moved on the sheet: C1, C10, C2, C3, C4, C5, C6, C7, C8, C9, J1, J2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
