File: pcb/power/power.kicad_pcb (KiCad board)
At the start: 2 copper layers, 226 x 89 mm, 282 parts, among them Q1 IPT015N10N5, Q10 IPT015N10N5, Q11 IPT015N10N5, Q12 IPT015N10N5, Q2 IPT015N10N5, Q3 IPT015N10N5, Q4 IPT015N10N5, Q5 IPT015N10N5, Q6 IPT015N10N5, Q7 IPT015N10N5, Q8 IPT015N10N5, Q9 IPT015N10N5

Commit message: Semifinish power and bulk
Parts:
- removed REF** (x205): C_1206_3216Metric, Capacitor_SMD:C_1206_3216Metric
- removed REF** (x9): PinHeader_2x01_P2.00mm_Vertical_SMD, Connector_PinHeader_2.00mm:PinHeader_2x01_P2.00mm_Vertical_SMD
- removed REF** (x3): SOIC-8_3.9x4.9mm_P1.27mm, Package_SO:SOIC-8_3.9x4.9mm_P1.27mm
- removed REF** (x19): MountingHole_5.3mm_M5_DIN965_Pad_TopBottom, MountingHole:MountingHole_5.3mm_M5_DIN965_Pad_TopBottom
- removed REF**: LQFP-48_7x7mm_P0.5mm, Package_QFP:LQFP-48_7x7mm_P0.5mm
- removed REF** (x18): C_Radial_D12.5mm_H25.0mm_P5.00mm, Capacitor_THT:C_Radial_D12.5mm_H25.0mm_P5.00mm
- removed REF** (x9): PinSocket_2x01_P2.00mm_Vertical_SMD, Connector_PinSocket_2.00mm:PinSocket_2x01_P2.00mm_Vertical_SMD
- added C1: 100n, Capacitor_SMD:C_0402_1005Metric, F.Cu at (92.3, 81.2)
- added C10: 2u2, Capacitor_SMD:C_1206_3216Metric, F.Cu at (32.5, 63.0)
- added C11: 100n, Capacitor_SMD:C_0402_1005Metric, F.Cu at (92.3, 59.2)
- added C12: 2u2, Capacitor_SMD:C_1206_3216Metric, F.Cu at (32.5, 59.0)
- added C13: 2u2, Capacitor_SMD:C_1206_3216Metric, F.Cu at (32.5, 56.8)
- added C14: 2u2, Capacitor_SMD:C_1206_3216Metric, F.Cu at (32.5, 54.5)
- added C15: 2u2, Capacitor_SMD:C_1206_3216Metric, F.Cu at (32.5, 52.2)
- added C16: 2u2, Capacitor_SMD:C_1206_3216Metric, F.Cu at (32.5, 50.0)
- added C17: 2u2, Capacitor_SMD:C_1206_3216Metric, F.Cu at (32.5, 47.8)
- added C18: 2u2, Capacitor_SMD:C_1206_3216Metric, F.Cu at (32.5, 45.5)
- added C19: 2u2, Capacitor_SMD:C_1206_3216Metric, F.Cu at (32.5, 43.2)
- added C2: 2u2, Capacitor_SMD:C_1206_3216Metric, F.Cu at (32.5, 81.0)
- added C20: 2u2, Capacitor_SMD:C_1206_3216Metric, F.Cu at (32.5, 41.0)
- added C21: 100n, Capacitor_SMD:C_0402_1005Metric, F.Cu at (92.3, 37.2)
- added C22: 2u2, Capacitor_SMD:C_1206_3216Metric, F.Cu at (32.5, 37.0)
- added C23: 2u2, Capacitor_SMD:C_1206_3216Metric, F.Cu at (32.5, 34.8)
- added C24: 2u2, Capacitor_SMD:C_1206_3216Metric, F.Cu at (32.5, 32.5)
- added C25: 2u2, Capacitor_SMD:C_1206_3216Metric, F.Cu at (32.5, 30.2)
- added C26: 2u2, Capacitor_SMD:C_1206_3216Metric, F.Cu at (32.5, 28.0)
- added C27: 2u2, Capacitor_SMD:C_1206_3216Metric, F.Cu at (32.5, 25.8)
- added C28: 2u2, Capacitor_SMD:C_1206_3216Metric, F.Cu at (32.5, 23.5)
- added C29: 2u2, Capacitor_SMD:C_1206_3216Metric, F.Cu at (32.5, 21.2)
- added C3: 2u2, Capacitor_SMD:C_1206_3216Metric, F.Cu at (32.5, 78.8)
- added C30: 2u2, Capacitor_SMD:C_1206_3216Metric, F.Cu at (32.5, 19.0)
- added C4: 2u2, Capacitor_SMD:C_1206_3216Metric, F.Cu at (32.5, 76.5)
- added C5: 2u2, Capacitor_SMD:C_1206_3216Metric, F.Cu at (32.5, 74.2)
- added C6: 2u2, Capacitor_SMD:C_1206_3216Metric, F.Cu at (32.5, 72.0)
- added C7: 2u2, Capacitor_SMD:C_1206_3216Metric, F.Cu at (32.5, 69.8)
- added C8: 2u2, Capacitor_SMD:C_1206_3216Metric, F.Cu at (32.5, 67.5)
- added C9: 2u2, Capacitor_SMD:C_1206_3216Metric, F.Cu at (32.5, 65.2)
- added J1: Conn_02x01, Connector_PinHeader_1.27mm:PinHeader_2x01_P1.27mm_Vertical_SMD, F.Cu at (63.0, 81.8)
- added J2: Conn_02x03_Odd_Even, Connector_PinHeader_1.27mm:PinHeader_2x03_P1.27mm_Vertical_SMD, F.Cu at (87.0, 80.5)
- added J3: Conn_02x01, Connector_PinHeader_1.27mm:PinHeader_2x01_P1.27mm_Vertical_SMD, F.Cu at (63.0, 59.8)
- added J4: Conn_02x03_Odd_Even, Connector_PinHeader_1.27mm:PinHeader_2x03_P1.27mm_Vertical_SMD, F.Cu at (87.0, 58.5)
- added J5: Conn_02x01, Connector_PinHeader_1.27mm:PinHeader_2x01_P1.27mm_Vertical_SMD, F.Cu at (63.0, 37.8)
- added J6: Conn_02x03_Odd_Even, Connector_PinHeader_1.27mm:PinHeader_2x03_P1.27mm_Vertical_SMD, F.Cu at (87.0, 36.5)
- added R7: 1m, Resistor_SMD:R_2512_6332Metric, F.Cu at (89.0, 29.8)
- added R8: 1m, Resistor_SMD:R_2512_6332Metric, F.Cu at (89.0, 25.8)
- added R9: 1m, Resistor_SMD:R_2512_6332Metric, F.Cu at (89.0, 21.8)
- added U1: INA181, Package_TO_SOT_SMD:SOT-23-6, F.Cu at (92.5, 79.0)
- added U2: INA181, Package_TO_SOT_SMD:SOT-23-6, F.Cu at (92.5, 57.0)
- added U3: INA181, Package_TO_SOT_SMD:SOT-23-6, F.Cu at (92.5, 35.0)
- Q1, Q10, Q11, Q12, Q2, Q3, Q4, Q5, Q6, Q7, Q8, Q9: value IPT015N10N5 -> IPT015N10NF2S
- R1, R2, R3, R4, R5, R6: footprint Resistor_SMD:R_4020_10251Metric -> Resistor_SMD:R_2512_6332Metric
- moved Q2 69.5 mm to (51.8, 66.8)
- moved Q5 66.6 mm to (51.8, 55.2)
- moved Q10 66.4 mm to (51.8, 22.8)
- moved R5 65.7 mm to (89.0, 47.8)
- moved R3 60.5 mm to (89.0, 65.8)
- moved Q4 52.4 mm to (75.8, 66.8)
- moved R1 47.6 mm to (89.0, 73.8)
- moved R2 46.8 mm to (89.0, 69.8)
- moved R4 45.9 mm to (89.0, 51.8)
- moved R6 44.4 mm to (89.0, 43.8)
- moved Q6 44.2 mm to (51.8, 44.8)
- moved Q12 44.1 mm to (75.8, 22.8)
- moved Q7 43.9 mm to (75.8, 55.2)
- moved Q9 43.5 mm to (51.8, 33.2)
- moved Q1 43.4 mm to (51.8, 77.2)
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Connections:
- net GND renamed GNDPWR
- Q1 pad 1: /Phase2/GH -> /Phase1/GH
- Q1 pad 2: /Phase2/OUT -> /Phase1/PH
- Q1 pad 3: VDD -> VBUS
- Q10 pad 1: /Phase3/GL -> /Phase3/GH
- Q10 pad 2: Net-(Q10-S) -> /Phase3/PH
- Q10 pad 3: /Phase3/OUT -> VBUS
- Q11 pad 1: /Phase3/GH -> /Phase3/GL
- Q11 pad 2: /Phase3/OUT -> /Phase3/SH
- Q11 pad 3: VDD -> /Phase3/PH
- Q12 pad 2: Net-(Q10-S) -> /Phase3/SH
- Q12 pad 3: /Phase3/OUT -> /Phase3/PH
- Q2 pad 1: /Phase2/GL -> /Phase1/GH
- Q2 pad 2: Net-(Q2-S) -> /Phase1/PH
- Q2 pad 3: /Phase2/OUT -> VBUS
- Q3 pad 1: /Phase2/GH -> /Phase1/GL
- Q3 pad 2: /Phase2/OUT -> /Phase1/SH
- Q3 pad 3: VDD -> /Phase1/PH
- Q4 pad 1: /Phase2/GL -> /Phase1/GL
- Q4 pad 2: Net-(Q2-S) -> /Phase1/SH
- Q4 pad 3: /Phase2/OUT -> /Phase1/PH
- Q5 pad 1: /Phase1/GL -> /Phase2/GH
- Q5 pad 2: Net-(Q5-S) -> /Phase2/PH
- Q5 pad 3: /Phase1/OUT -> VBUS
- Q6 pad 1: /Phase1/GH -> /Phase2/GH
- Q6 pad 2: /Phase1/OUT -> /Phase2/PH
- Q6 pad 3: VDD -> VBUS
- Q7 pad 1: /Phase1/GL -> /Phase2/GL
- Q7 pad 2: Net-(Q5-S) -> /Phase2/SH
- Q7 pad 3: /Phase1/OUT -> /Phase2/PH
- Q8 pad 1: /Phase1/GH -> /Phase2/GL
- Q8 pad 2: /Phase1/OUT -> /Phase2/SH
- Q8 pad 3: VDD -> /Phase2/PH
- Q9 pad 2: /Phase3/OUT -> /Phase3/PH
- Q9 pad 3: VDD -> VBUS
- R1 pad 1: Net-(Q5-S) -> /Phase1/SH
- R2 pad 1: Net-(Q2-S) -> /Phase1/SH
- R3 pad 1: Net-(Q10-S) -> /Phase1/SH
- R4 pad 1: Net-(Q5-S) -> /Phase2/SH
- R5 pad 1: Net-(Q2-S) -> /Phase2/SH
- R6 pad 1: Net-(Q10-S) -> /Phase2/SH
Routing:
- net /Phase1/GH: track 14.3 -> 0.00 mm
- net /Phase3/GH: track 11.8 -> 0.00 mm
- added copper zone on F.Cu, net /Phase1/PH
- added copper zone on F.Cu, net /Phase1/SH
- added copper zone on F.Cu, net /Phase2/PH
- added copper zone on F.Cu, net /Phase2/SH
- added copper zone on F.Cu, net /Phase3/PH
- added copper zone on F.Cu, net /Phase3/SH
- added copper zone on F.Cu, net GNDPWR
- added copper zone on F.Cu, net VBUS
Other:
- board size 226 x 89 mm -> 75 x 65 mm

Commit message: Save progress
Parts:
- J1, J3, J5: value Conn_02x01 -> Conn_02x02_Odd_Even; footprint Connector_PinHeader_1.27mm:PinHeader_2x01_P1.27mm_Vertical_SMD -> Connector_PinHeader_1.27mm:PinHeader_2x02_P1.27mm_Vertical_SMD
- moved J1 0.75 mm to (63.0, 81.0)
- moved J3 0.75 mm to (63.0, 59.0)
- moved J5 0.75 mm to (63.0, 37.0)
Connections:
- J1 pad 1: /Phase1/GH -> /Phase1/PH
- J3 pad 1: /Phase2/GH -> /Phase2/PH
- J5 pad 1: /Phase3/GH -> /Phase3/PH

Commit message: Update shunts
Parts:
- removed R1, R2, R3, R4, R5, R6, R7, R8, R9: 1m, Resistor_SMD:R_2512_6332Metric
- added REF**: R_4020_10251Metric, Resistor_SMD:R_4020_10251Metric, F.Cu at (88.8, 31.0)
- added REF**: R_4020_10251Metric, Resistor_SMD:R_4020_10251Metric, F.Cu at (88.9, 41.4)
- added REF**: R_4020_10251Metric, Resistor_SMD:R_4020_10251Metric, F.Cu at (88.8, 69.0)
- added REF**: R_4020_10251Metric, Resistor_SMD:R_4020_10251Metric, F.Cu at (88.8, 20.2)
- added REF**: R_4020_10251Metric, Resistor_SMD:R_4020_10251Metric, F.Cu at (88.7, 74.5)
- added REF**: R_4020_10251Metric, Resistor_SMD:R_4020_10251Metric, F.Cu at (88.9, 52.3)
- added REF**: R_4020_10251Metric, Resistor_SMD:R_4020_10251Metric, F.Cu at (88.8, 63.5)
- added REF**: R_4020_10251Metric, Resistor_SMD:R_4020_10251Metric, F.Cu at (88.8, 25.6)
- added REF**: R_4020_10251Metric, Resistor_SMD:R_4020_10251Metric, F.Cu at (88.9, 46.8)
Routing:
- removed copper zone on F.Cu, net /Phase1/SH
- removed copper zone on F.Cu, net /Phase2/SH
- removed copper zone on F.Cu, net /Phase3/SH

Commit message: Finish rev 1
Parts:
- removed REF** (x9): R_4020_10251Metric, Resistor_SMD:R_4020_10251Metric
- added R1: 1m, User_Footprints:R_Shunt_3921, F.Cu at (88.8, 74.6)
- added R2: 1m, User_Footprints:R_Shunt_3921, F.Cu at (88.8, 69.1)
- added R3: 1m, User_Footprints:R_Shunt_3921, F.Cu at (88.8, 63.6)
- added R4: 1m, User_Footprints:R_Shunt_3921, F.Cu at (88.8, 52.9)
- added R5: 1m, User_Footprints:R_Shunt_3921, F.Cu at (88.8, 47.4)
- added R6: 1m, User_Footprints:R_Shunt_3921, F.Cu at (88.8, 41.9)
- added R7: 1m, User_Footprints:R_Shunt_3921, F.Cu at (88.8, 31.3)
- added R8: 1m, User_Footprints:R_Shunt_3921, F.Cu at (88.8, 25.8)
- added R9: 1m, User_Footprints:R_Shunt_3921, F.Cu at (88.8, 20.3)
- Q1, Q10, Q11, Q12, Q2, Q3, Q4, Q5, Q6, Q7, Q8, Q9: value IPT015N10NF2S -> SP010N01BGHTO
- moved C21 0.59 mm to (91.8, 37.6), turned to 0 degrees
- moved U3 0.58 mm to (92.5, 35.6)
- moved J1 0.50 mm to (62.5, 81.0)
- moved J2 0.50 mm to (86.5, 80.5)
- moved J3 0.50 mm to (62.5, 59.0)
- moved J4 0.50 mm to (86.5, 58.5)
- moved J5 0.50 mm to (62.5, 37.0)
- moved J6 0.50 mm to (86.5, 36.5)
- moved C1 0.40 mm to (92.0, 80.9), turned to 0 degrees
- moved C11 0.37 mm to (91.9, 59.2), turned to 0 degrees
- moved U2 0.26 mm to (92.5, 57.3)
- moved U1 0.18 mm to (92.7, 78.9)
- moved Q10 0.07 mm to (51.8, 22.8)
- moved Q12 0.07 mm to (75.8, 22.8)
- moved Q1 0.07 mm to (51.8, 77.3)
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Connections:
- C1 pad 1: VCC -> /Phase1/3V3
- C1 pad 2: GND -> /Phase1/AGND
- C10 pad 2: GNDPWR -> GNDRET
- C11 pad 1: VCC -> /Phase2/3V3
- C11 pad 2: GND -> /Phase2/AGND
- C12 pad 2: GNDPWR -> GNDRET
- C13 pad 2: GNDPWR -> GNDRET
- C14 pad 2: GNDPWR -> GNDRET
- C15 pad 2: GNDPWR -> GNDRET
- C16 pad 2: GNDPWR -> GNDRET
- C17 pad 2: GNDPWR -> GNDRET
- C18 pad 2: GNDPWR -> GNDRET
- C19 pad 2: GNDPWR -> GNDRET
- C2 pad 2: GNDPWR -> GNDRET
- C20 pad 2: GNDPWR -> GNDRET
- C21 pad 1: VCC -> /Phase3/3V3
- C21 pad 2: GND -> /Phase3/AGND
- C22 pad 2: GNDPWR -> GNDRET
- C23 pad 2: GNDPWR -> GNDRET
- C24 pad 2: GNDPWR -> GNDRET
- C25 pad 2: GNDPWR -> GNDRET
- C26 pad 2: GNDPWR -> GNDRET
- C27 pad 2: GNDPWR -> GNDRET
- C28 pad 2: GNDPWR -> GNDRET
- C29 pad 2: GNDPWR -> GNDRET
- C3 pad 2: GNDPWR -> GNDRET
- C30 pad 2: GNDPWR -> GNDRET
- C4 pad 2: GNDPWR -> GNDRET
- C5 pad 2: GNDPWR -> GNDRET
- C6 pad 2: GNDPWR -> GNDRET
- C7 pad 2: GNDPWR -> GNDRET
- C8 pad 2: GNDPWR -> GNDRET
- C9 pad 2: GNDPWR -> GNDRET
- J2 pad 2: VCC -> /Phase1/3V3
- J2 pad 4: GND -> /Phase1/AGND
- J4 pad 2: VCC -> /Phase2/3V3
- J4 pad 4: GND -> /Phase2/AGND
- J6 pad 2: VCC -> /Phase3/3V3
- J6 pad 4: GND -> /Phase3/AGND
- U1 pad 2: GND -> /Phase1/AGND
- U1 pad 6: VCC -> /Phase1/3V3
- U2 pad 2: GND -> /Phase2/AGND
- U2 pad 6: VCC -> /Phase2/3V3
- U3 pad 2: GND -> /Phase3/AGND
- U3 pad 6: VCC -> /Phase3/3V3
Routing:
- net /Phase2/GH: track 0.00 -> 21.9 mm
- net /Phase1/GH: track 0.00 -> 21.9 mm
- net /Phase3/GH: track 0.00 -> 21.7 mm
- net /Phase1/GL: track 0.00 -> 17.8 mm
- net /Phase2/GL: track 0.00 -> 17.7 mm
- net /Phase3/GL: track 0.00 -> 17.7 mm
- net GNDPWR: track 0.00 -> 12.9 mm
- net /Phase3/AGND: track 0.00 -> 9.87 mm
- net /Phase1/AGND: track 0.00 -> 9.82 mm
- net /Phase2/AGND: track 0.00 -> 9.66 mm
- net /Phase2/CUR: track 0.00 -> 8.28 mm
- net /Phase3/VREF: track 0.00 -> 7.88 mm
- net /Phase1/VREF: track 0.00 -> 7.67 mm
- net /Phase2/VREF: track 0.00 -> 7.60 mm
- net /Phase3/CUR: track 0.00 -> 7.09 mm
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- added copper zone on F.Cu, net /Phase1/SH
- added copper zone on F.Cu, net /Phase2/SH
- added copper zone on F.Cu, net /Phase3/SH
- added copper zone on F.Cu, net GNDRET
