File: pcb/logic/logic.kicad_sch (KiCad schematic)
At the start: 1 part, among them U4 STM32G431C6Tx

Commit message: Finish rev 1
Parts:
- removed U4: STM32G431C6Tx, Package_QFP:LQFP-48_7x7mm_P0.5mm, symbol MCU_ST_STM32G4:STM32G431C6Tx
- added C13, C19, C41, C42, C43, C44, C46, C47, C48, C49, C50, C52, C54, C55: 100n, Capacitor_SMD:C_0402_1005Metric, symbol Device:C
- added C17: 220p, Capacitor_SMD:C_0402_1005Metric, symbol Device:C
- added C18: 10n, Capacitor_SMD:C_0402_1005Metric, symbol Device:C
- added C20, C40, C57: 22u, Capacitor_SMD:C_1206_3216Metric, symbol Device:C
- added C21, C45, C56, C59: 4u7, Capacitor_SMD:C_0805_2012Metric, symbol Device:C
- added C51, C53: 10p, Capacitor_SMD:C_0402_1005Metric, symbol Device:C
- added C58: 1n, Capacitor_SMD:C_0402_1005Metric, symbol Device:C
- added D1: LED, LED_SMD:LED_0603_1608Metric, symbol Device:LED
- added FB1: 120, Inductor_SMD:L_0603_1608Metric, symbol Device:FerriteBead
- added J10, J7, J8: Conn_01x02, User_Footprints:1x02_2.00mm_Solder, symbol Connector_Generic:Conn_01x02
- added J11: Conn_01x06, User_Footprints:1x06_2.00mm_Solder, symbol Connector_Generic:Conn_01x06
- added J9: Conn_ARM_SWD_TagConnect_TC2030-NL, Connector:Tag-Connect_TC2030-IDC-NL_2x03_P1.27mm_Vertical, symbol Connector:Conn_ARM_SWD_TagConnect_TC2030-NL
- added JP1: SolderJumper_3_Open, SolderJumper-3_P1.3mm_Open_RoundedPad1.0x1.5mm, symbol Jumper:SolderJumper_3_Open
- added L2: 4u7, Inductor_SMD:L_TechFuse_SL0420, symbol Device:L
- added R10, R12, R14, R29, R31, R35, R36: 2k2, Resistor_SMD:R_0402_1005Metric, symbol Device:R
- added R11, R13, R30, R33, R34: 33k, Resistor_SMD:R_0402_1005Metric, symbol Device:R
- added R24, R25: 51, Resistor_SMD:R_0805_2012Metric, symbol Device:R
- added R32: 330, Resistor_SMD:R_0402_1005Metric, symbol Device:R
- added R39: 12k, Resistor_SMD:R_0402_1005Metric, symbol Device:R
- added TH4: 10k, Resistor_SMD:R_0402_1005Metric, symbol Device:Thermistor
- added U14: JW5017S, Package_TO_SOT_SMD:SOT-23-6, symbol User_Symbols:JW5017S
- added U4: AMS1117-3.3, Package_TO_SOT_SMD:SOT-223-3_TabPin2, symbol Regulator_Linear:AMS1117-3.3
- added U5: STM32G473CBTx, Package_QFP:LQFP-48_7x7mm_P0.5mm, symbol MCU_ST_STM32G4:STM32G473CBTx
- added U6: SP485E, Package_SO:JEITA_SOIC-8_3.9x4.9mm_P1.27mm, symbol User_Symbols:SP485E
- added Y1: 16MHz, Crystal:Crystal_SMD_3225-4Pin_3.2x2.5mm, symbol Device:Crystal_GND24
Connections:
- new net: R11.2, R13.1
- new net: R33.1, R34.2
- new net +15V: C56.1, J8.1 (Pin_1), R30.1, U14.5 (VIN)
- new net +3V3: C20.1, C41.1, C45.1, C46.1, C47.1, C48.1, C49.1, FB1.1, J9.1 (VCC), JP1.3 (B), R10.1, R31.1, U4.2 (VO), U5.1 (VBAT), U5.24 (VDD), U5.36 (VDD), U5.48 (VDD)
- new net +3V3A: C54.1, C58.1, C59.1, FB1.2, U5.20 (VREF+), U5.21 (VDDA)
- new net +5V: C21.1, C40.1, C42.1, C52.1, C57.1, JP1.1 (A), L2.2, R39.1, U4.3 (VI), U6.8 (VCC)
- new net ACUR: U5.17 (PB1)
- new net AINH: U5.30 (PA8)
- new net AINL: U5.33 (PA11)
- new net ASNS: U5.27 (PB13)
- new net ATEMP: U5.9 (PA1)
- new net BCUR: U5.28 (PB14)
- new net BINH: U5.31 (PA9)
- new net BINL: U5.34 (PA12)
- new net BOOT0: R36.1, U5.45 (PB8)
- new net BSNS: U5.26 (PB12)
- new net BT: C55.1, U14.1 (BST)
- new net BTEMP: U5.8 (PA0)
- new net BUSF: C17.1, R13.2, R14.1, U5.15 (PA7)
- new net BUSL: C18.1, R12.1, R33.2, U5.10 (PA2)
- new net CCUR: U5.13 (PA5)
- new net CINH: U5.32 (PA10)
- new net CINL: U5.46 (PB9)
- new net CSNS: U5.14 (PA6)
- new net CTEMP: U5.16 (PB0)
- new net DEN: U5.2 (PC13), U6.3 (DE)
- new net EN: R30.2, U14.4 (EN)
- new net EVCC: C43.1, J11.1 (Pin_1), JP1.2 (C)
- new net FB: R29.1, R39.2, U14.3 (FB)
- new net FLTC: U5.39 (PA15)
- new net FLTV: U5.22 (PB10)
- new net GND: C13.2, C17.2, C18.2, C19.1, C20.2, C21.2, C40.2, C41.2, C42.2, C43.2, C44.2, C45.2, C46.2, C47.2, C48.2, C49.2, C50.2, C51.1, C52.2, C53.1, C54.2, C56.2, C57.2, C58.2, C59.2, D1.1 (K), J11.2 (Pin_2), J11.5 (Pin_5), J7.1 (Pin_1), J9.5 (GND), R12.2, R14.2, R29.2, R36.2, TH4.2, U14.2 (GND), U4.1 (GND), U5.12 (PA4), U5.18 (PB2), U5.19 (VSSA), U5.23 (VSS), U5.29 (PB15), U5.35 (VSS), U5.47 (VSS), U6.5 (GND), Y1.2, Y1.4
- new net LED: R35.1, U5.3 (PC14)
- new net LR: D1.2 (A), R35.2
- new net MTEMP: C44.1, J7.2 (Pin_2), R31.2, U5.11 (PA3)
- new net NRST: C50.1, J9.3 (~{RESET}), U5.7 (PG10)
- new net QA: J11.3 (Pin_3), U5.41 (PB4)
- new net QB: J11.4 (Pin_4), U5.42 (PB5)
- new net QZ: J11.6 (Pin_6), U5.40 (PB3)
- new net REN: U5.4 (PC15), U6.2 (~{RE})
- new net RSA: J10.2 (Pin_2), R24.1, U6.6 (A)
- new net RSB: J10.1 (Pin_1), R25.2, U6.7 (B)
- new net RX: U5.44 (PB7), U6.1 (RO)
- new net SPL: C19.2, R24.2, R25.1
- new net SW: C55.2, L2.1, U14.6 (SW)
- new net SWCLK: J9.4 (SWCLK), U5.38 (PA14)
- new net SWDIO: J9.2 (SWDIO), U5.37 (PA13)
- new net TEMP: C13.1, R10.2, TH4.1, U5.25 (PB11)
- new net TX: U5.43 (PB6), U6.4 (DI)
- new net VBUS: J8.2 (Pin_2), R11.1, R34.1
- new net XTALI: C51.2, U5.5 (PF0), Y1.1
- new net XTALO: R32.2, U5.6 (PF1)
- new net XTALR: C53.2, R32.1, Y1.3
- no-connect marks 0 -> 1
Other:
- sheet Phase1 ports: added CUR, FLTC, FLTV, INH, INL, TEMP, VSNS; removed none
- sheet Phase2 ports: added CUR, FLTC, FLTV, INH, INL, TEMP, VSNS; removed none
- sheet Phase3 ports: added CUR, FLTC, FLTV, INH, INL, TEMP, VSNS; removed none
- note added: "360khz"
- note added: "5.1V"
- note added: "7khz"
- note added: "Board Temp"
- note added: "Buck 15V -> 5V"
- note added: "Bus Monitor"
- note added: "LDO 5V -> 3.3V"
- note added: "MCU"
- note added: "Motor Encoder + Temp"
- note added: "Phases"
- note added: "Power"
- note added: "RS-485"
